File: deckPCB/deckPCB.kicad_sch (KiCad schematic)
At the start: 0 parts

Commit message: deckPCB Changes
Parts:
- added U1: RP2040, RP2040:QFN40P700X700X90-57N, symbol RP2040:RP2040
- added U2: W25Q128JVE, Package_SON:WSON-8-1EP_8x6mm_P1.27mm_EP3.4x4.3mm, symbol Memory_Flash:W25Q128JVE
- added X1, X2: DF40HC_3.0_-100DS-0.4V_58, DF40HC_3.0_-100DS-0.4V_58:HRS_DF40HC_3.0_-100DS-0.4V_58, symbol DF40HC_3.0_-100DS-0.4V_58:DF40HC_3.0_-100DS-0.4V_58
Connections:
- new net DVDD: U1.23 (DVDD), U1.50 (DVDD)
- new net IOVDD: U1.1 (IOVDD), U1.10 (IOVDD), U1.22 (IOVDD), U1.33 (IOVDD), U1.42 (IOVDD), U1.49 (IOVDD)
Changed lines of the file:
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@@
 	(generator_version "10.0")
 	(paper "A4")
-	(sheet_instances
-		(path "/"
-			(page "1")
-		)
-	)
-	(embedded_fonts no)
-)

Commit message: donr
Parts:
- added J1: USB_C_Receptacle_USB2.0_16P, symbol Connector:USB_C_Receptacle_USB2.0_16P
- added L1: L, symbol Device:L
- added SW1, SW10, SW11, SW12, SW13, SW14, SW15, SW2, SW3, SW4, SW5, SW6, SW7, SW8, SW9: SW_Push, symbol Switch:SW_Push
- added U3: IP5306, IP5306:SOP127P600X165-9N, symbol IP5306:IP5306
- added U4: AMS1117-3.3, Package_TO_SOT_SMD:SOT-223-3_TabPin2, symbol Regulator_Linear:AMS1117-3.3
Connections:
- new net: J1.A1 (GND), J1.A12 (GND), J1.B1 (GND), J1.B12 (GND)
- new net: J1.A4 (VBUS), J1.A9 (VBUS), J1.B4 (VBUS), J1.B9 (VBUS)
Other:
- note added: "(Right Angle Switch)"
- note added: "K silver hall joystick yet to be added"
- moved on the sheet: U1, U2, X1, X2

Commit message: somethign
Parts:
- added C1, C2: C, symbol Device:C
- added J2: Conn_01x06_Pin, symbol Connector:Conn_01x06_Pin
- added LS1, LS2: Speaker, symbol Device:Speaker
- added U5: PAM8403DR, PAM8403DR:SOIC127P605X150-16N, symbol PAM8403DR:PAM8403DR
Other:
- note added: "Audio & Storage"
- note added: "The Controller Inputs"
- note added: "The Core Processing"
- note added: "The Power Section"
- moved on the sheet: J1, L1, SW1, SW10, SW11, SW12, SW13, SW14, SW15, SW2, SW3, SW4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
Changed lines of the file:
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@@
 	(generator "eeschema")
 	(generator_version "10.0")
-	(paper "A4")
+	(paper "A3")

Commit message: Finishing with the passives.
Parts:
- added C10, C11, C12, C13, C14, C15, C16, C17, C18, C19, C20, C3, C4, C5, C6, C7, C8, C9: C, symbol Device:C
- added R1, R2, R3, R4, R5, R6, R7, R8: R, symbol Device:R
Other:
- moved on the sheet: C1, C2, J1, J2, L1, LS1, LS2, U3, U4, U5

Commit message: hall symbol in the schematic
Parts:
- added JS1, JS2: (no value), symbol ArxDeck_Custom:K-Silver_JH16
Other:
- note removed: "K silver hall joystick yet to be added"
- moved on the sheet: C14, C15, C16, C17, C18, C19, C20, J2, LS1, LS2, R8, SW1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

Commit message: wiring_power
Parts:
- added BT1: Battery_Cell, symbol Device:Battery_Cell
Connections:
- net IOVDD is gone; now on net DVDD: U1.1 (IOVDD), U1.10 (IOVDD), U1.22 (IOVDD), U1.33 (IOVDD), U1.42 (IOVDD), U1.49 (IOVDD)
- net DVDD: now also C2.1, U1.44 (VREG_VIN), U4.2 (VO)
- net GND: now reaches J1.A1 (GND), J1.A12 (GND), J1.B1 (GND), J1.B12 (GND)
- net GND: now also U1.57 (GND), U3.9 (POWERPAD), U4.1 (GND), BT1.2 (-)
- net VBUS_5V: now reaches J1.A4 (VBUS), J1.A9 (VBUS), J1.B4 (VBUS), J1.B9 (VBUS)
- net CC1: now reaches J1.A5 (CC1)
- net CC2: now reaches J1.B5 (CC2)
- net CPC1: now reaches L1.2
- net CPC1: now also C1.1, U3.8 (VOUT)
- net BATT+: now reaches U3.6 (BAT)
- net BATT+: now also BT1.1 (+)
- net SW_NODE: now reaches U3.7 (SW)
Other:
- moved on the sheet: C1, C10, C11, C12, C13, C14, C15, C16, C17, C18, C19, C2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
